File: unexpected_grizzly.kicad_pcb (KiCad board)
At the start: 2 copper layers, 49.5 x 49.5 mm, 30 parts, among them P1 USB, P2 GPIO, P3 FTDI, SW1 RESET, U1 NCP1117ST33T3G, U2 ESP-12

Commit message: Correction to USB pinout. Other tidy-ups.
Parts:
- removed the REF** at (158.8, 93.7)
- moved C2 1.33 mm to (140.3, 91.9)
- moved C1 1.30 mm to (140.2, 88.0), turned to 270 degrees
- moved U1 1.13 mm to (134.0, 89.9)
Routing:
- net GND: track 113.0 -> 99.3 mm
- net +3V3: track 98.8 -> 92.3 mm
- net +5V: track 27.9 -> 29.1 mm
- net GPIO16: track 24.7 -> 24.1 mm

Commit message: Final V1
Parts:
- moved P1 0.32 mm to (126.5, 99.8)
Routing:
- net GND: track 99.3 -> 98.7 mm
Changed lines of the file:
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@@
     (thickness 1.6)
     (drawings 20)
-    (tracks 295)
+    (tracks 297)
     (zones 0)
     (modules 29)
@@
     (mod_text_size 1 1)
     (mod_text_width 0.15)
-    (pad_size 3.6576 2.032)
-    (pad_drill 0)
+    (pad_size 3.1 3.1)
+    (pad_drill 3.1)
     (pad_to_mask_clearance 0)
     (aux_axis_origin 0 0)
     (visible_elements FFFFFF7F)
     (pcbplotparams
-      (layerselection 0x00030_80000001)
-      (usegerberextensions false)
+      (layerselection 0x010f0_80000001)
+      (usegerberextensions true)
       (excludeedgelayer true)
       (linewidth 0.100000)
@@
       (outputformat 1)
       (mirror false)
-      (drillshape 1)
+      (drillshape 0)
       (scaleselection 1)
-      (outputdirectory ""))
+      (outputdirectory output))
   )
   (net 0 "")
@@
     (tags "capacitor 0805")
     (attr smd)
-    (fp_text reference C1 (at 2.4055 -0.012 360) (layer F.SilkS)
+    (fp_text reference C1 (at -2.47 -0.05 360) (layer F.SilkS)
       (effects (font (size 1 1) (thickness 0.15)))
     )
@@
     (tags "capacitor 0805")
     (attr smd)
-    (fp_text reference C2 (at 2.6555 -0.0415 360) (layer F.SilkS)
+    (fp_text reference C2 (at 2.54 -0.04 360) (layer F.SilkS)
       (effects (font (size 1 1) (thickness 0.15)))
     )
@@
     (descr "Through hole pin header")
     (tags "pin header")
-    (fp_text reference JP1 (at 0.086 -2.57 450) (layer F.SilkS)
+    (fp_text reference JP1 (at 0.086 -2.57 270) (layer F.SilkS) hide
       (effects (font (size 1 1) (thickness 0.15)))
     )
@@
     (descr "Through hole pin header")
     (tags "pin header")
-    (fp_text reference P3 (at 0 15.113 180) (layer F.SilkS)
+    (fp_text reference P3 (at 0 15.113 180) (layer F.SilkS) hide
       (effects (font (size 1 1) (thickness 0.15)))
     )
@@
     )
     (fp_circle (center 0 0) (end 3 0) (layer F.Fab) (width 0.15))
-    (pad "" np_thru_hole circle (at 0 0) (size 3.1 3.1) (drill 3.1) (layers *.Cu))
+    (pad "" thru_hole circle (at 0 0) (size 3.1 3.1) (drill 3.1) (layers *.Cu *.Mask))
   )
   (module timhawes:MountingHole_M3+ (layer F.Cu)
@@
     )
     (fp_circle (center 0 0) (end 3 0) (layer F.Fab) (width 0.15))
-    (pad "" np_thru_hole circle (at 0 0) (size 3.1 3.1) (drill 3.1) (layers *.Cu))
+    (pad "" thru_hole circle (at 0 0) (size 3.1 3.1) (drill 3.1) (layers *.Cu *.Mask))
   )
   (module timhawes:MountingHole_M3+ (layer F.Cu)
@@
     )
     (fp_circle (center 0 0) (end 3 0) (layer F.Fab) (width 0.15))
-    (pad "" np_thru_hole circle (at 0 0) (size 3.1 3.1) (drill 3.1) (layers *.Cu))
+    (pad "" thru_hole circle (at 0 0) (size 3.1 3.1) (drill 3.1) (layers *.Cu *.Mask))
   )
   (module timhawes:MountingHole_M3+ (layer F.Cu)
@@
     )
     (fp_circle (center 0 0) (end 3 0) (layer F.Fab) (width 0.15))
-    (pad "" np_thru_hole circle (at 0 0) (size 3.1 3.1) (drill 3.1) (layers *.Cu))
+    (pad "" thru_hole circle (at 0 0) (size 3.1 3.1) (drill 3.1) (layers *.Cu *.Mask))
   )
   (module timhawes:Matrix_Row_19 (layer F.Cu)
@@
   )
   (module timhawes:FCI_10104110_0001LF (layer F.Cu)
-    (at 126.873 99.822 270)
-    (fp_text reference P1 (at 4 -3.7 270) (layer F.SilkS)
+    (at 126.55 99.81 270)
+    (fp_text reference P1 (at 2.64 -2.05 270) (layer F.SilkS)
       (effects (font (size 1 1) (thickness 0.15)))
     )
@@
   (gr_arc (start 171.45 125.73) (end 174.625 125.73) (angle 90) (layer Edge.Cuts) (width 0.2))
   (segment (start 174.625 128.905) (end 174.625 79.375) (width 0.25) (layer Dwgs.User) (net 0))
+  (segment (start 131.386799 98.826799) (end 131.082 98.522) (width 0.3048) (layer F.Cu) (net 1))
+  (segment (start 127 106.68) (end 131.811201 101.868799) (width 0.3048) (layer F.Cu) (net 1))
+  (segment (start 131.811201 99.251201) (end 131.386799 98.826799) (width 0.3048) (layer F.Cu) (net 1))
+  (segment (start 131.811201 101.868799) (end 131.811201 99.251201) (width 0.3048) (layer F.Cu) (net 1))
   (segment (start 136.25 88.55) (end 131.082 93.718) (width 0.3048) (layer B.Cu) (net 1))
   (segment (start 131.082 93.718) (end 131.082 98.522) (width 0.3048) (layer B.Cu) (net 1))
   (via (at 131.082 98.522) (size 0.6096) (drill 0.3048) (layers F.Cu B.Cu) (net 1))
-  (segment (start 127 106.68) (end 127.434846 106.68) (width 0.3048) (layer F.Cu) (net 1))
-  (segment (start 131.791201 102.323645) (end 131.791201 99.231201) (width 0.3048) (layer F.Cu) (net 1))
-  (segment (start 127.434846 106.68) (end 131.791201 102.323645) (width 0.3048) (layer F.Cu) (net 1))
-  (segment (start 131.791201 99.231201) (end 131.082 98.522) (width 0.3048) (layer F.Cu) (net 1))
   (segment (start 131.082 98.522) (end 129.723 98.522) (width 0.3048) (layer F.Cu) (net 1))
   (segment (start 137.254 87.654) (end 137.146 87.654) (width 0.3048) (layer F.Cu) (net 1))
@@
   (segment (start 137.254 87.654) (end 137.076 87.654) (width 0.3048) (layer F.Cu) (net 1))
   (segment (start 127.01 106.67) (end 127 106.68) (width 0.3048) (layer B.Cu) (net 1))
-  (segment (start 131.08 100.258948) (end 131.08 100.69) (width 0.3048) (layer B.Cu) (net 2))
-  (segment (start 133.543747 97.795201) (end 131.08 100.258948) (width 0.3048) (layer B.Cu) (net 2))
-  (segment (start 136.601479 97.795201) (end 133.543747 97.795201) (width 0.3048) (layer B.Cu) (net 2))
-  (segment (start 136.906278 98.1) (end 136.601479 97.795201) (width 0.3048) (layer B.Cu) (net 2))
+  (segment (start 129.54 106.68) (end 130.6 105.62) (width 0.3048) (layer B.Cu) (net 2))
+  (segment (start 130.6 105.62) (end 130.6 101.15) (width 0.3048) (layer B.Cu) (net 2))
+  (segment (start 130.6 101.15) (end 130.645201 101.104799) (width 0.3048) (layer B.Cu) (net 2))
+  (segment (start 130.645201 101.104799) (end 130.95 100.8) (width 0.3048) (layer B.Cu) (net 2))
+  (segment (start 131.254799 100.495201) (end 130.95 100.8) (width 0.3048) (layer B.Cu) (net 2))
+  (segment (start 130.628 101.122) (end 130.645201 101.104799) (width 0.3048) (layer F.Cu) (net 2))
+  (segment (start 133.65 98.1) (end 131.254799 100.495201) (width 0.3048) (layer B.Cu) (net 2))
+  (segment (start 136.906278 98.1) (end 133.65 98.1) (width 0.3048) (layer B.Cu) (net 2))
+  (segment (start 130.645201 101.104799) (end 130.95 100.8) (width 0.3048) (layer F.Cu) (net 2))
+  (segment (start 129.723 101.122) (end 130.628 101.122) (width 0.3048) (layer F.Cu) (net 2))
+  (via (at 130.95 100.8) (size 0.6096) (drill 0.3048) (layers F.Cu B.Cu) (net 2))
   (segment (start 138.54 93.63) (end 136.906278 95.263722) (width 0.3048) (layer B.Cu) (net 2))
   (segment (start 136.906278 95.263722) (end 136.906278 98.1) (width 0.3048) (layer B.Cu) (net 2))
@@
   (segment (start 137.254 92.226) (end 137.762 92.226) (width 0.3048) (layer F.Cu) (net 2))
   (segment (start 139.92 92.87) (end 139.79 92.87) (width 0.3048) (layer F.Cu) (net 2))
-  (segment (start 129.54 106.68) (end 131.08 105.14) (width 0.3048) (layer B.Cu) (net 2))
-  (segment (start 131.08 105.14) (end 131.08 100.69) (width 0.3048) (layer B.Cu) (net 2))
-  (segment (start 129.723 101.122) (end 130.648 101.122) (width 0.3048) (layer F.Cu) (net 2))
-  (segment (start 130.648 101.122) (end 131.08 100.69) (width 0.3048) (layer F.Cu) (net 2))
-  (via (at 131.08 100.69) (size 0.6096) (drill 0.3048) (layers F.Cu B.Cu) (net 2))
   (segment (start 166.88 99.3) (end 168.21 99.3) (width 0.3048) (layer B.Cu) (net 2))
   (segment (start 168.21 99.3) (end 170.51 101.6) (width 0.3048) (layer B.Cu) (net 2))
@@
     (polygon
       (pts
-        (xy 125.222 94.361) (xy 128.397 94.361) (xy 128.397 105.029) (xy 125.095 105.029) (xy 125.095 94.361)
+        (xy 127.67 94.51) (xy 127.67 105.06) (xy 125.095 105.06) (xy 125.095 94.51)
       )
     )
@@
     (polygon
       (pts
-        (xy 125.106723 85.6) (xy 135.74 85.6) (xy 135.74 96.67) (xy 128.76 96.67) (xy 128.76 94.01)
-        (xy 125.106723 94.01)
+        (xy 125.1 85.6) (xy 135.65 85.6) (xy 135.65 95.8) (xy 128 95.8) (xy 128 94.2)
+        (xy 125.1 94.2)
       )
     )
